Commit message: Fixed some issues but explotes in gazebo

File: champ_description/urdf/spot/spot.urdf.xacro (robot description, xacro)
@@ -19,4 +19,10 @@
     <xacro:include filename="spot_leg.urdf.xacro" />
     <xacro:include filename="camera.xacro" />
+    <!-- Dummy base link without inertia -->
+    <link name="$(arg prefix)base_footprint" />
+    <joint name="$(arg prefix)base_footprint_joint" type="fixed">
+    <parent link="$(arg prefix)base_footprint" />
+    <child link="$(arg prefix)base_link" />
+    </joint>
     <link name="$(arg prefix)base_link">
         <visual>
@@ -59,6 +65,6 @@
     <xacro:empty_link name="$(arg prefix)rear_rail" />
     <xacro:fixed_joint name="rear_rail_joint" parent="$(arg prefix)body" child="$(arg prefix)rear_rail" xyz="-0.223 0 0.0805" />
+    <xacro:spot_leg leg_name="front_right" prefix="$(arg prefix)" />
     <xacro:spot_leg leg_name="front_left" prefix="$(arg prefix)" />
-    <xacro:spot_leg leg_name="front_right" prefix="$(arg prefix)" />
     <xacro:spot_leg leg_name="rear_left" prefix="$(arg prefix)" />
     <xacro:spot_leg leg_name="rear_right" prefix="$(arg prefix)" />
@@ -143,5 +149,5 @@
                 <remapping>odom:=odom/ground_truth</remapping>
             </ros>
-            <body_name>base_link</body_name>
+            <body_name>body</body_name>
             <update_rate>20</update_rate>
             <xyz_offset>0 0 0</xyz_offset>

File: champ_description/urdf/spot/spot_leg.urdf.xacro (robot description, xacro)
@@ -157,5 +157,5 @@
             </actuator>
         </transmission>
-        <ros2_control name="GazeboSystem" type="system">
+        <ros2_control name="${leg_name}_GazeboSystem" type="system">
             <hardware>
                 <plugin>gazebo_ros2_control/GazeboSystem</plugin>

Commit message: enable rviz odom estimation

File: champ_description/urdf/spot/spot.urdf.xacro (robot description, xacro)
@@ -12,6 +12,6 @@
     <xacro:arg name="simulate_cameras" default="False" />
     <xacro:arg name="simulate_imu" default="False" />
-    <xacro:arg name="body_color_r" default="${str(234/255.0)}" />
-    <xacro:arg name="body_color_g" default="${str(167/255.0)}" />
+    <xacro:arg name="body_color_r" default="${str(234.0/255.0)}" />
+    <xacro:arg name="body_color_g" default="${str(167.0/255.0)}" />
     <xacro:arg name="body_color_b" default="0" />
     <xacro:include filename="utils.xacro" />
@@ -20,9 +20,9 @@
     <xacro:include filename="camera.xacro" />
     <!-- Dummy base link without inertia -->
-    <link name="$(arg prefix)base_footprint" />
+    <!-- <link name="$(arg prefix)base_footprint" />
     <joint name="$(arg prefix)base_footprint_joint" type="fixed">
     <parent link="$(arg prefix)base_footprint" />
     <child link="$(arg prefix)base_link" />
-    </joint>
+    </joint> -->
     <link name="$(arg prefix)base_link">
         <visual>

Commit message: Fix body model

File: champ_description/urdf/spot/spot.urdf.xacro (robot description, xacro)
@@ -28,10 +28,10 @@
         <visual>
             <geometry>
-                <mesh filename="$(find champ_description)/meshes/spot/body.dae" />
+                <mesh filename="file://$(find champ_description)/meshes/spot/body.dae" />
             </geometry>
         </visual>
         <collision>
             <geometry>
-                <mesh filename="$(find champ_description)/meshes/spot/body_collision.stl" />
+                <mesh filename="file://$(find champ_description)/meshes/spot/body_collision.stl" />
             </geometry>
         </collision>

Commit message: checking URDF

File: champ_description/urdf/spot/spot.urdf.xacro (robot description, xacro)
@@ -19,11 +19,5 @@
     <xacro:include filename="spot_leg.urdf.xacro" />
     <xacro:include filename="camera.xacro" />
-    <!-- Dummy base link without inertia -->
-    <!-- <link name="$(arg prefix)base_footprint" />
-    <joint name="$(arg prefix)base_footprint_joint" type="fixed">
-    <parent link="$(arg prefix)base_footprint" />
-    <child link="$(arg prefix)base_link" />
-    </joint> -->
-    <link name="$(arg prefix)base_link">
+    <link name="$(arg prefix)body">
         <visual>
             <geometry>
@@ -32,13 +26,38 @@
         </visual>
         <collision>
+            <origin rpy="0 0 0" xyz="0 0 0"/>
             <geometry>
-                <mesh filename="file://$(find champ_description)/meshes/spot/body_collision.stl" />
+                <!-- <mesh filename="file://$(find champ_description)/meshes/spot/body_collision.stl" /> -->
+                <box size="${base_length} ${base_width} ${base_height}"/>
             </geometry>
         </collision>
         <inertial>
-            <mass value="${base_mass}" />
-            <inertia ixx="${(1/12) * base_mass * (base_width * base_width + base_height * base_height)}" ixy="0.0" ixz="0.0" iyy="${(1/12) * base_mass * (base_length * base_length + base_height * base_height)}" iyz="0.0" izz="${(1/12) * base_mass * (base_length * base_length + base_width * base_width)}" />
+            <mass value="${base_mass}"/>
+            <inertia ixx="${(1/12) * base_mass * (base_width * base_width + base_height * base_height)}" ixy="0.0" ixz="0.0"
+                        iyy="${(1/12) * base_mass * (base_length * base_length + base_height * base_height)}" iyz="0.0"
+                        izz="${(1/12) * base_mass * (base_length * base_length + base_width * base_width)}" />
         </inertial>
     </link>
+    <link name="$(arg prefix)base_link"/>
+    <joint name="$(arg prefix)base_link_joint" type="fixed">
+        <origin xyz="0 0 0" rpy="0 0 0" />
+        <parent link="$(arg prefix)base_link" />
+        <child link="$(arg prefix)body" />
+    </joint>
+    <gazebo reference="$(arg prefix)base_link">
+        <kp>400000.0</kp>
+        <kd>1.0</kd>
+        <mu1>0.8</mu1>
+        <mu2>0.8</mu2>
+        <maxVel>0.0</maxVel>
+        <minDepth>0.002</minDepth>
+    </gazebo>
+    <link name="$(arg prefix)base_footprint">
+    </link>
+    <joint name="$(arg prefix)base_footprint_joint" type="fixed">
+        <origin xyz="0 0 -0.5" rpy="0 0 0"/>
+        <parent link="$(arg prefix)base_link"/>
+        <child link="$(arg prefix)base_footprint"/>
+    </joint>
     <link name="$(arg prefix)battery">
         <visual>
@@ -59,6 +78,4 @@
     <xacro:solid_color_link_material link="$(arg prefix)battery" r="$(arg body_color_r)" g="$(arg body_color_g)" b="$(arg body_color_b)" />
     <xacro:fixed_joint name="battery_joint" parent="$(arg prefix)base_link" child="$(arg prefix)battery" xyz="0 0 -0.03" />
-    <xacro:empty_link name="$(arg prefix)body" />
-    <xacro:fixed_joint name="base_link_joint" parent="$(arg prefix)base_link" child="$(arg prefix)body" />
     <xacro:empty_link name="$(arg prefix)front_rail" />
     <xacro:fixed_joint name="front_rail_joint" parent="$(arg prefix)body" child="$(arg prefix)front_rail" xyz="0.223 0 0.0805" />
@@ -149,5 +166,5 @@
                 <remapping>odom:=odom/ground_truth</remapping>
             </ros>
-            <body_name>body</body_name>
+            <body_name>$(arg prefix)base_link</body_name>
             <update_rate>20</update_rate>
             <xyz_offset>0 0 0</xyz_offset>

File: champ_description/urdf/spot/spot_leg.urdf.xacro (robot description, xacro)
@@ -5,4 +5,6 @@
     <xacro:arg name="leg_mu1" default="1.0" />
     <xacro:arg name="leg_mu2" default="1.0" />
+    <xacro:arg name="leg_maxVel" default="0.0" />
+    <xacro:arg name="leg_minDepth" default="0.002" />
     <xacro:arg name="leg_fdir1" default="" />
     <xacro:arg name="max_knee_effort" default="80" />
@@ -35,14 +37,24 @@
                 </geometry>
             </visual>
-            <collision>
+            <!-- <collision>
                 <geometry>
                     <mesh filename="file://$(find champ_description)/meshes/spot/${leg_name}_hip_collision.stl" />
                 </geometry>
-            </collision>
+            </collision> -->
             <inertial>
                 <mass value="${hip_mass}" />
-                <inertia ixx="${(1/12) * hip_mass * (hip_width * hip_width + hip_height * hip_height)}" ixy="0.0" ixz="0.0" iyy="${(1/12) * hip_mass * (hip_length * hip_length + hip_height * hip_height)}" iyz="0.0" izz="${(1/12) * hip_mass * (hip_length * hip_length + hip_width * hip_width)}" />
+                <inertia ixx="${(1/12) * hip_mass * (hip_width * hip_width + hip_height * hip_height)}" ixy="0.0" ixz="0.0"
+                            iyy="${(1/12) * hip_mass * (hip_length * hip_length + hip_height * hip_height)}" iyz="0.0"
+                            izz="${(1/12) * hip_mass * (hip_length * hip_length + hip_width * hip_width)}" />
             </inertial>
         </link>
+        <gazebo reference="${prefix}${leg_name}_hip">
+            <kp>$(arg leg_kp)</kp>
+            <kd>$(arg leg_kd)</kd>
+            <mu1>$(arg leg_mu1)</mu1>
+            <mu2>$(arg leg_mu2)</mu2>
+            <mu2>$(arg leg_maxVel)</mu2>
+            <mu2>$(arg leg_minDepth)</mu2>
+        </gazebo>
         <joint name="${leg_name}_hip_x" type="revolute">
             <origin xyz="${base_to_hip_xyz}" rpy="0 0 0" />
@@ -60,6 +72,8 @@
             </visual>
             <collision>
-                <geometry>
-                    <mesh filename="file://$(find champ_description)/meshes/spot/${leg_name}_upper_leg_collision.stl" />
+                <origin rpy="0 0 0" xyz="0 0 ${-0.25*upper_leg_height}"/>
+                <geometry>
+                    <!-- <mesh filename="file://$(find champ_description)/meshes/spot/${leg_name}_upper_leg_collision.stl" /> -->
+                    <cylinder radius="${0.6*upper_leg_width}" length="${0.8*upper_leg_height}"/>
                 </geometry>
             </collision>
@@ -67,7 +81,17 @@
                 <origin xyz="0 0 -0.14" rpy="0 0 0" />
                 <mass value="${upper_leg_mass}" />
-                <inertia ixx="${(1/12) * upper_leg_mass * (upper_leg_width * upper_leg_width + upper_leg_height * upper_leg_height)}" ixy="0.0" ixz="0.0" iyy="${(1/12) * upper_leg_mass * (upper_leg_length * upper_leg_length + upper_leg_height * upper_leg_height)}" iyz="0.0" izz="${(1/12) * upper_leg_mass * (upper_leg_length * upper_leg_length + upper_leg_width * upper_leg_width)}" />
+                <inertia ixx="${(1/12) * upper_leg_mass * (upper_leg_width * upper_leg_width + upper_leg_height * upper_leg_height)}" ixy="0.0" ixz="0.0"
+                            iyy="${(1/12) * upper_leg_mass * (upper_leg_length * upper_leg_length + upper_leg_height * upper_leg_height)}" iyz="0.0"
+                            izz="${(1/12) * upper_leg_mass * (upper_leg_length * upper_leg_length + upper_leg_width * upper_leg_width)}" />
             </inertial>
         </link>
+        <gazebo reference="${prefix}${leg_name}_upper_leg">
+            <kp>$(arg leg_kp)</kp>
+            <kd>$(arg leg_kd)</kd>
+            <mu1>$(arg leg_mu1)</mu1>
+            <mu2>$(arg leg_mu2)</mu2>
+            <mu2>$(arg leg_maxVel)</mu2>
+            <mu2>$(arg leg_minDepth)</mu2>
+        </gazebo>
         <joint name="${leg_name}_hip_y" type="revolute">
             <origin xyz="${hip_to_upper_leg_xyz}" rpy="0 0 0" />
@@ -85,12 +109,8 @@
             </visual>
             <collision>
-                <geometry>
-                    <mesh filename="file://$(find champ_description)/meshes/spot/${leg_name}_lower_leg_collision.stl" scale="0.82 0.97 0.98" />
-                </geometry>
-            </collision>
-            <collision>
-                <origin xyz="0 0 -${lower_leg_to_foot_z - 0.04 + 0.003}" />
-                <geometry>
-                    <sphere radius="0.04" />
+                <origin rpy="0 0 0" xyz="0 0 ${-0.35*lower_leg_height}"/>
+                <geometry>
+                    <!-- <mesh filename="file://$(find champ_description)/meshes/spot/${leg_name}_lower_leg_collision.stl" scale="0.82 0.97 0.98" /> -->
+                    <cylinder radius="${lower_leg_length}" length="${0.6*lower_leg_height}"/>
                 </geometry>
             </collision>
@@ -98,5 +118,7 @@
                 <origin xyz="0 0 -0.16" rpy="0 0 0" />
                 <mass value="${lower_leg_mass}" />
-                <inertia ixx="${(1/12) * lower_leg_mass * (lower_leg_width * lower_leg_width + lower_leg_height * lower_leg_height)}" ixy="0.0" ixz="0.0" iyy="${(1/12) * lower_leg_mass * (lower_leg_length * lower_leg_length + lower_leg_height * lower_leg_height)}" iyz="0.0" izz="${(1/12) * lower_leg_mass * (lower_leg_length * lower_leg_length + lower_leg_width * lower_leg_width)}" />
+                <inertia ixx="${(1/12) * lower_leg_mass * (lower_leg_width * lower_leg_width + lower_leg_height * lower_leg_height)}" ixy="0.0" ixz="0.0"
+                         iyy="${(1/12) * lower_leg_mass * (lower_leg_length * lower_leg_length + lower_leg_height * lower_leg_height)}" iyz="0.0"
+                         izz="${(1/12) * lower_leg_mass * (lower_leg_length * lower_leg_length + lower_leg_width * lower_leg_width)}" />
             </inertial>
         </link>
@@ -106,4 +128,6 @@
             <mu1>$(arg leg_mu1)</mu1>
             <mu2>$(arg leg_mu2)</mu2>
+            <mu2>$(arg leg_maxVel)</mu2>
+            <mu2>$(arg leg_minDepth)</mu2>
             <xacro:if value="${'$(arg leg_fdir1)' != ''}">
                 <fdir1>$(arg leg_fdir1)</fdir1>
@@ -124,8 +148,28 @@
             <dynamics damping="10.0" friction="100.0" />
         </joint>
-        <xacro:empty_link name="${prefix}${leg_name}_ee" />
-        <xacro:fixed_joint name="${leg_name}_foot" parent="${prefix}${leg_name}_lower_leg" child="${prefix}${leg_name}_ee" xyz="0 0 -${lower_leg_to_foot_z}" />
+        <!-- <xacro:empty_link name="${prefix}${leg_name}_ee" /> -->
+        <link name="${prefix}${leg_name}_ee">
+            <collision name="${prefix}${leg_name}_ee_collision">
+                <origin rpy="0 0 0" xyz="0 0 ${lower_leg_length}"/>
+                <geometry>
+                    <sphere radius="${lower_leg_length}"/>
+                </geometry>
+            </collision>
+        </link>
+        <joint name="${prefix}${leg_name}_foot" type="fixed">
+            <parent link="${prefix}${leg_name}_lower_leg" />
+            <child link="${prefix}${leg_name}_ee" />
+            <origin xyz="0 0 -${lower_leg_to_foot_z}" rpy="0 0 0" />
+        </joint>
+        <gazebo reference="${prefix}${leg_name}_ee">
+            <kp>$(arg leg_kp)</kp>
+            <kd>$(arg leg_kd)</kd>
+            <mu1>$(arg leg_mu1)</mu1>
+            <mu2>$(arg leg_mu2)</mu2>
+            <mu2>$(arg leg_maxVel)</mu2>
+            <mu2>$(arg leg_minDepth)</mu2>
+        </gazebo>
         <!-- Not actually used now, but doesn't hurt to have it here ready for future use with ros_ign_control. -->
-        <transmission name="${leg_name}_hip_x_trans">
+        <!-- <transmission name="${leg_name}_hip_x_trans">
             <type>transmission_interface/SimpleTransmission</type>
             <joint name="${leg_name}_hip_x">
@@ -156,5 +200,5 @@
                 <mechanicalReduction>1</mechanicalReduction>
             </actuator>
-        </transmission>
+        </transmission> -->
         <ros2_control name="${leg_name}_GazeboSystem" type="system">
             <hardware>

Commit message: tests

File: champ_description/urdf/spot/spot.urdf.xacro (robot description, xacro)
@@ -45,5 +45,5 @@
         <child link="$(arg prefix)body" />
     </joint>
-    <gazebo reference="$(arg prefix)base_link">
+    <!-- <gazebo reference="$(arg prefix)base_link">
         <kp>400000.0</kp>
         <kd>1.0</kd>
@@ -52,5 +52,5 @@
         <maxVel>0.0</maxVel>
         <minDepth>0.002</minDepth>
-    </gazebo>
+    </gazebo> -->
     <link name="$(arg prefix)base_footprint">
     </link>

File: champ_description/urdf/spot/spot_leg.urdf.xacro (robot description, xacro)
@@ -1,8 +1,12 @@
 <?xml version="1.0"?>
 <robot xmlns:xacro="http://ros.org/wiki/xacro">
-    <xacro:arg name="leg_kp" default="1e+07" />
-    <xacro:arg name="leg_kd" default="100.0" />
-    <xacro:arg name="leg_mu1" default="1.0" />
-    <xacro:arg name="leg_mu2" default="1.0" />
+    <!-- <xacro:arg name="leg_kp" default="1e+07" /> -->
+    <!-- <xacro:arg name="leg_kd" default="100.0" /> -->
+    <!-- <xacro:arg name="leg_mu1" default="1.0" />
+    <xacro:arg name="leg_mu2" default="1.0" /> -->
+    <xacro:arg name="leg_kp" default="40000.0" />
+    <xacro:arg name="leg_kd" default="1.0" />
+    <xacro:arg name="leg_mu1" default="0.8" />
+    <xacro:arg name="leg_mu2" default="0.8" />
     <xacro:arg name="leg_maxVel" default="0.0" />
     <xacro:arg name="leg_minDepth" default="0.002" />
@@ -49,5 +53,5 @@
             </inertial>
         </link>
-        <gazebo reference="${prefix}${leg_name}_hip">
+        <!-- <gazebo reference="${prefix}${leg_name}_hip">
             <kp>$(arg leg_kp)</kp>
             <kd>$(arg leg_kd)</kd>
@@ -56,5 +60,5 @@
             <mu2>$(arg leg_maxVel)</mu2>
             <mu2>$(arg leg_minDepth)</mu2>
-        </gazebo>
+        </gazebo> -->
         <joint name="${leg_name}_hip_x" type="revolute">
             <origin xyz="${base_to_hip_xyz}" rpy="0 0 0" />
@@ -63,5 +67,5 @@
             <child link="${prefix}${leg_name}_hip" />
             <limit effort="$(arg max_hip_x_effort)" velocity="$(arg max_hip_x_velocity)" lower="-0.78539816339744827899" upper="0.78539816339744827899" />
-            <dynamics damping="10.0" friction="100.0" />
+            <dynamics damping="10.0" friction="1e+07" />
         </joint>
         <link name="${prefix}${leg_name}_upper_leg">
@@ -86,5 +90,5 @@
             </inertial>
         </link>
-        <gazebo reference="${prefix}${leg_name}_upper_leg">
+        <!-- <gazebo reference="${prefix}${leg_name}_upper_leg">
             <kp>$(arg leg_kp)</kp>
             <kd>$(arg leg_kd)</kd>
@@ -93,5 +97,5 @@
             <mu2>$(arg leg_maxVel)</mu2>
             <mu2>$(arg leg_minDepth)</mu2>
-        </gazebo>
+        </gazebo> -->
         <joint name="${leg_name}_hip_y" type="revolute">
             <origin xyz="${hip_to_upper_leg_xyz}" rpy="0 0 0" />
@@ -100,5 +104,5 @@
             <child link="${prefix}${leg_name}_upper_leg" />
             <limit effort="$(arg max_hip_y_effort)" velocity="$(arg max_hip_y_velocity)" lower="-0.89884456477707963539" upper="2.2951079663725435509" />
-            <dynamics damping="10.0" friction="100.0" />
+            <dynamics damping="10.0" friction="1e+07" />
         </joint>
         <link name="${prefix}${leg_name}_lower_leg">
@@ -124,10 +128,10 @@
         </link>
         <gazebo reference="${prefix}${leg_name}_lower_leg">
-            <kp>$(arg leg_kp)</kp>
-            <kd>$(arg leg_kd)</kd>
-            <mu1>$(arg leg_mu1)</mu1>
-            <mu2>$(arg leg_mu2)</mu2>
-            <mu2>$(arg leg_maxVel)</mu2>
-            <mu2>$(arg leg_minDepth)</mu2>
+            <!-- <kp>$(arg leg_kp)</kp>
+            <kd>$(arg leg_kd)</kd>
+            <mu1>$(arg leg_mu1)</mu1>
+            <mu2>$(arg leg_mu2)</mu2>
+            <mu2>$(arg leg_maxVel)</mu2>
+            <mu2>$(arg leg_minDepth)</mu2> -->
             <xacro:if value="${'$(arg leg_fdir1)' != ''}">
                 <fdir1>$(arg leg_fdir1)</fdir1>
@@ -146,5 +150,5 @@
             <child link="${prefix}${leg_name}_lower_leg" />
             <limit effort="$(arg max_knee_effort)" velocity="$(arg max_knee_velocity)" lower="-2.7929" upper="-0.254801" />
-            <dynamics damping="10.0" friction="100.0" />
+            <dynamics damping="10.0" friction="1e+07" />
         </joint>
         <!-- <xacro:empty_link name="${prefix}${leg_name}_ee" /> -->
@@ -161,6 +165,8 @@
             <child link="${prefix}${leg_name}_ee" />
             <origin xyz="0 0 -${lower_leg_to_foot_z}" rpy="0 0 0" />
-        </joint>
-        <gazebo reference="${prefix}${leg_name}_ee">
+            <limit effort="$(arg max_knee_effort)" velocity="$(arg max_knee_velocity)" lower="-2.7929" upper="-0.254801" />
+            <dynamics damping="10.0" friction="1e+07" />
+        </joint>
+        <!-- <gazebo reference="${prefix}${leg_name}_ee">
             <kp>$(arg leg_kp)</kp>
             <kd>$(arg leg_kd)</kd>
@@ -169,5 +175,5 @@
             <mu2>$(arg leg_maxVel)</mu2>
             <mu2>$(arg leg_minDepth)</mu2>
-        </gazebo>
+        </gazebo> -->
         <!-- Not actually used now, but doesn't hurt to have it here ready for future use with ros_ign_control. -->
         <!-- <transmission name="${leg_name}_hip_x_trans">
@@ -210,5 +216,7 @@
                     <param name="max">${pi}</param>
                 </command_interface>
-                <state_interface name="position" />
+                <state_interface name="position" >
+                    <param name="initial_value">0.0</param>
+                </state_interface>
                 <state_interface name="velocity" />
                 <state_interface name="effort" />
@@ -219,5 +227,7 @@
                     <param name="max">${pi}</param>
                 </command_interface>
-                <state_interface name="position" />
+                <state_interface name="position" >
+                    <param name="initial_value">1.4880125522613525</param>
+                </state_interface>
                 <state_interface name="velocity" />
                 <state_interface name="effort" />
@@ -228,5 +238,7 @@
                     <param name="max">${pi}</param>
                 </command_interface>
-                <state_interface name="position" />
+                <state_interface name="position" >
+                    <param name="initial_value">-2.51871919631958</param>
+                </state_interface>
                 <state_interface name="velocity" />
                 <state_interface name="effort" />
