Commit message: cleaning

File: champ_description/urdf/spot/spot.urdf.xacro (robot description, xacro)
@@ -45,12 +45,4 @@
         <child link="$(arg prefix)body" />
     </joint>
-    <!-- <gazebo reference="$(arg prefix)base_link">
-        <kp>400000.0</kp>
-        <kd>1.0</kd>
-        <mu1>0.8</mu1>
-        <mu2>0.8</mu2>
-        <maxVel>0.0</maxVel>
-        <minDepth>0.002</minDepth>
-    </gazebo> -->
     <link name="$(arg prefix)base_footprint">
     </link>

File: champ_description/urdf/spot/spot_leg.urdf.xacro (robot description, xacro)
@@ -1,12 +1,12 @@
 <?xml version="1.0"?>
 <robot xmlns:xacro="http://ros.org/wiki/xacro">
-    <!-- <xacro:arg name="leg_kp" default="1e+07" /> -->
-    <!-- <xacro:arg name="leg_kd" default="100.0" /> -->
-    <!-- <xacro:arg name="leg_mu1" default="1.0" />
-    <xacro:arg name="leg_mu2" default="1.0" /> -->
-    <xacro:arg name="leg_kp" default="40000.0" />
+    <xacro:arg name="leg_kp" default="1e+07" />  <!--contact stiffness-->
+    <xacro:arg name="leg_kd" default="1.0" /> <!--damping-->
+    <xacro:arg name="leg_mu1" default="1e+07" />
+    <xacro:arg name="leg_mu2" default="0.8" />
+    <!-- <xacro:arg name="leg_kp" default="400000.0" />
     <xacro:arg name="leg_kd" default="1.0" />
     <xacro:arg name="leg_mu1" default="0.8" />
-    <xacro:arg name="leg_mu2" default="0.8" />
+    <xacro:arg name="leg_mu2" default="0.8" /> -->
     <xacro:arg name="leg_maxVel" default="0.0" />
     <xacro:arg name="leg_minDepth" default="0.002" />
@@ -18,4 +18,6 @@
     <xacro:arg name="max_hip_y_effort" default="80" />
     <xacro:arg name="max_hip_y_velocity" default="15" />
+    <xacro:arg name="damping" default="0.0" />
+    <xacro:arg name="friction" default="1.0e+07" />
     <xacro:macro name="spot_leg" params="leg_name prefix">
         <xacro:if value="${leg_name == 'front_left'}">
@@ -53,13 +55,5 @@
             </inertial>
         </link>
-        <!-- <gazebo reference="${prefix}${leg_name}_hip">
-            <kp>$(arg leg_kp)</kp>
-            <kd>$(arg leg_kd)</kd>
-            <mu1>$(arg leg_mu1)</mu1>
-            <mu2>$(arg leg_mu2)</mu2>
-            <mu2>$(arg leg_maxVel)</mu2>
-            <mu2>$(arg leg_minDepth)</mu2>
-        </gazebo> -->
-        <joint name="${leg_name}_hip_x" type="revolute">
+        <joint name="${prefix}${leg_name}_hip_x" type="revolute">
             <origin xyz="${base_to_hip_xyz}" rpy="0 0 0" />
             <axis xyz="1 0 0" />
@@ -67,5 +61,5 @@
             <child link="${prefix}${leg_name}_hip" />
             <limit effort="$(arg max_hip_x_effort)" velocity="$(arg max_hip_x_velocity)" lower="-0.78539816339744827899" upper="0.78539816339744827899" />
-            <dynamics damping="10.0" friction="1e+07" />
+            <dynamics damping="$(arg damping)" friction="$(arg friction)" />
         </joint>
         <link name="${prefix}${leg_name}_upper_leg">
@@ -90,13 +84,5 @@
             </inertial>
         </link>
-        <!-- <gazebo reference="${prefix}${leg_name}_upper_leg">
-            <kp>$(arg leg_kp)</kp>
-            <kd>$(arg leg_kd)</kd>
-            <mu1>$(arg leg_mu1)</mu1>
-            <mu2>$(arg leg_mu2)</mu2>
-            <mu2>$(arg leg_maxVel)</mu2>
-            <mu2>$(arg leg_minDepth)</mu2>
-        </gazebo> -->
-        <joint name="${leg_name}_hip_y" type="revolute">
+        <joint name="${prefix}${leg_name}_hip_y" type="revolute">
             <origin xyz="${hip_to_upper_leg_xyz}" rpy="0 0 0" />
             <axis xyz="0 1 0" />
@@ -104,5 +90,5 @@
             <child link="${prefix}${leg_name}_upper_leg" />
             <limit effort="$(arg max_hip_y_effort)" velocity="$(arg max_hip_y_velocity)" lower="-0.89884456477707963539" upper="2.2951079663725435509" />
-            <dynamics damping="10.0" friction="1e+07" />
+            <dynamics damping="$(arg damping)" friction="$(arg friction)" />
         </joint>
         <link name="${prefix}${leg_name}_lower_leg">
@@ -127,11 +113,35 @@
             </inertial>
         </link>
-        <gazebo reference="${prefix}${leg_name}_lower_leg">
-            <!-- <kp>$(arg leg_kp)</kp>
+        <joint name="${prefix}${leg_name}_knee" type="revolute">
+            <origin xyz="${upper_leg_to_lower_leg_x} 0 -${upper_leg_to_lower_leg_z}" rpy="0 0 0" />
+            <axis xyz="0 1 0" />
+            <parent link="${prefix}${leg_name}_upper_leg" />
+            <child link="${prefix}${leg_name}_lower_leg" />
+            <limit effort="$(arg max_knee_effort)" velocity="$(arg max_knee_velocity)" lower="-2.7929" upper="-0.254801" />
+            <dynamics damping="$(arg damping)" friction="$(arg friction)" />
+        </joint>
+        <!-- <xacro:empty_link name="${prefix}${leg_name}_ee" /> -->
+        <link name="${prefix}${leg_name}_ee">
+            <collision name="${prefix}${leg_name}_ee_collision">
+                <origin rpy="0 0 0" xyz="0 0 ${lower_leg_length}"/>
+                <geometry>
+                    <sphere radius="${lower_leg_length}"/>
+                </geometry>
+            </collision>
+        </link>
+        <joint name="${prefix}${leg_name}_foot" type="fixed">
+            <parent link="${prefix}${leg_name}_lower_leg" />
+            <child link="${prefix}${leg_name}_ee" />
+            <origin xyz="0 0 -${lower_leg_to_foot_z}" rpy="0 0 0" />
+            <limit effort="$(arg max_knee_effort)" velocity="$(arg max_knee_velocity)" lower="-2.7929" upper="-0.254801" />
+            <dynamics damping="$(arg damping)" friction="$(arg friction)" />
+        </joint>
+        <gazebo reference="${prefix}${leg_name}_ee">
+            <kp>$(arg leg_kp)</kp>
             <kd>$(arg leg_kd)</kd>
             <mu1>$(arg leg_mu1)</mu1>
             <mu2>$(arg leg_mu2)</mu2>
-            <mu2>$(arg leg_maxVel)</mu2>
-            <mu2>$(arg leg_minDepth)</mu2> -->
+            <maxVel>$(arg leg_maxVel)</maxVel>
+            <minDepth>$(arg leg_minDepth)</minDepth>
             <xacro:if value="${'$(arg leg_fdir1)' != ''}">
                 <fdir1>$(arg leg_fdir1)</fdir1>
@@ -143,39 +153,34 @@
                 </contact>
             </sensor>
+            <maxContacts>1</maxContacts>
+            <minDepth>0.005</minDepth>
+            <gravity>true</gravity>
+            <collision name="${prefix}${leg_name}_ee_collision">
+                <geometry>
+                    <sphere>
+                        <!-- should be the same as surface_radius -->
+                        <radius>0.02175</radius>
+                    </sphere>
+                </geometry>
+            <surface>
+                <friction>
+                    <torsional>
+                        <coefficient>10</coefficient>
+                        <use_patch_radius>false</use_patch_radius>
+                        <!-- should be the same as collision sphere radius -->
+                        <surface_radius>0.02175</surface_radius>
+                        <patch_radius>0.01</patch_radius>
+                    </torsional>
+                </friction>
+                <contact>
+                    <poissons_ratio>0.5</poissons_ratio>
+                    <elastic_modulus>1e8</elastic_modulus>
+                </contact>
+            </surface>
+            </collision>
+            <material>Gazebo/Black</material>
         </gazebo>
-        <joint name="${leg_name}_knee" type="revolute">
-            <origin xyz="${upper_leg_to_lower_leg_x} 0 -${upper_leg_to_lower_leg_z}" rpy="0 0 0" />
-            <axis xyz="0 1 0" />
-            <parent link="${prefix}${leg_name}_upper_leg" />
-            <child link="${prefix}${leg_name}_lower_leg" />
-            <limit effort="$(arg max_knee_effort)" velocity="$(arg max_knee_velocity)" lower="-2.7929" upper="-0.254801" />
-            <dynamics damping="10.0" friction="1e+07" />
-        </joint>
-        <!-- <xacro:empty_link name="${prefix}${leg_name}_ee" /> -->
-        <link name="${prefix}${leg_name}_ee">
-            <collision name="${prefix}${leg_name}_ee_collision">
-                <origin rpy="0 0 0" xyz="0 0 ${lower_leg_length}"/>
-                <geometry>
-                    <sphere radius="${lower_leg_length}"/>
-                </geometry>
-            </collision>
-        </link>
-        <joint name="${prefix}${leg_name}_foot" type="fixed">
-            <parent link="${prefix}${leg_name}_lower_leg" />
-            <child link="${prefix}${leg_name}_ee" />
-            <origin xyz="0 0 -${lower_leg_to_foot_z}" rpy="0 0 0" />
-            <limit effort="$(arg max_knee_effort)" velocity="$(arg max_knee_velocity)" lower="-2.7929" upper="-0.254801" />
-            <dynamics damping="10.0" friction="1e+07" />
-        </joint>
-        <!-- <gazebo reference="${prefix}${leg_name}_ee">
-            <kp>$(arg leg_kp)</kp>
-            <kd>$(arg leg_kd)</kd>
-            <mu1>$(arg leg_mu1)</mu1>
-            <mu2>$(arg leg_mu2)</mu2>
-            <mu2>$(arg leg_maxVel)</mu2>
-            <mu2>$(arg leg_minDepth)</mu2>
-        </gazebo> -->
         <!-- Not actually used now, but doesn't hurt to have it here ready for future use with ros_ign_control. -->
-        <!-- <transmission name="${leg_name}_hip_x_trans">
+        <transmission name="${leg_name}_hip_x_trans">
             <type>transmission_interface/SimpleTransmission</type>
             <joint name="${leg_name}_hip_x">
@@ -206,5 +211,5 @@
                 <mechanicalReduction>1</mechanicalReduction>
             </actuator>
-        </transmission> -->
+        </transmission>
         <ros2_control name="${leg_name}_GazeboSystem" type="system">
             <hardware>
