Commit message: Starting changes to work with IGNITION

File: champ_description/urdf/spot/camera.xacro (robot description, xacro)
@@ -46,5 +46,13 @@
                         </lens>
                     </camera>
-                    <plugin filename="mono-camera-system" name="subt::MonoCameraSystem" />
+                    <plugin filename="libmono_camera_system.so" name="subt::MonoCameraSystem" >
+                     <!-- added by diya 8/30  -->
+                        <camera>
+                            <image_topic>camera/image_raw</image_topic>
+                            <camera_info_topic>camera/camera_info</camera_info_topic>
+                            <frame_name>camera_frame</frame_name>
+                            <update_rate>30.0</update_rate>
+                        </camera>
+                    </plugin>
                 </sensor>
                 <sensor name="${name}_depth" type="depth_camera">

File: champ_description/urdf/spot/spot.urdf.xacro (robot description, xacro)
@@ -12,6 +12,6 @@
     <xacro:arg name="simulate_cameras" default="False" />
     <xacro:arg name="simulate_imu" default="False" />
-    <xacro:arg name="body_color_r" default="${str(234.0/255.0)}" />
-    <xacro:arg name="body_color_g" default="${str(167.0/255.0)}" />
+    <xacro:arg name="body_color_r" default="${str(234/255.0)}" />
+    <xacro:arg name="body_color_g" default="${str(167/255.0)}" />
     <xacro:arg name="body_color_b" default="0" />
     <xacro:include filename="utils.xacro" />
@@ -45,11 +45,4 @@
         <child link="$(arg prefix)body" />
     </joint>
-    <link name="$(arg prefix)base_footprint">
-    </link>
-    <joint name="$(arg prefix)base_footprint_joint" type="fixed">
-        <origin xyz="0 0 -0.5" rpy="0 0 0"/>
-        <parent link="$(arg prefix)base_link"/>
-        <child link="$(arg prefix)base_footprint"/>
-    </joint>
     <link name="$(arg prefix)battery">
         <visual>
@@ -74,6 +67,6 @@
     <xacro:empty_link name="$(arg prefix)rear_rail" />
     <xacro:fixed_joint name="rear_rail_joint" parent="$(arg prefix)body" child="$(arg prefix)rear_rail" xyz="-0.223 0 0.0805" />
+    <xacro:spot_leg leg_name="front_left" prefix="$(arg prefix)" />
     <xacro:spot_leg leg_name="front_right" prefix="$(arg prefix)" />
-    <xacro:spot_leg leg_name="front_left" prefix="$(arg prefix)" />
     <xacro:spot_leg leg_name="rear_left" prefix="$(arg prefix)" />
     <xacro:spot_leg leg_name="rear_right" prefix="$(arg prefix)" />
@@ -152,19 +145,119 @@
     <xacro:spot_camera prefix="$(arg prefix)" name="back" simulate="$(arg simulate_cameras)" />
     <xacro:fixed_joint name="camera_back_j" parent="$(arg prefix)base_link" child="$(arg prefix)camera_back" xyz="-0.425 0 0.01" rpy="0 0.3 ${-pi}" />
-    <gazebo>
-        <plugin name="p3d_base_controller" filename="libgazebo_ros_p3d.so">
-            <ros>
-                <namespace></namespace>
-                <remapping>odom:=odom/ground_truth</remapping>
-            </ros>
-            <body_name>$(arg prefix)base_link</body_name>
-            <update_rate>20</update_rate>
-            <xyz_offset>0 0 0</xyz_offset>
-            <rpy_offset>0.0 0.0 0.0</rpy_offset>
-            <gaussian_noise>0.01</gaussian_noise>
-        </plugin>
-    </gazebo>
-    <gazebo>
-        <plugin name="gazebo_ros2_control" filename="libgazebo_ros2_control.so">
+    <!-- <ros2_control name="IgnitionSystem" type="system">
+        <hardware>
+            <plugin>ign_ros2_control/IgnitionSystem</plugin>
+        </hardware>
+        <joint name="front_left_hip_x">
+            <command_interface name="position">
+               <param name="min">-${pi}</param>
+                <param name="max">${pi}</param>
+            </command_interface>
+            <state_interface name="position" />
+            <state_interface name="velocity" />
+            <state_interface name="effort" />
+        </joint>
+        <joint name="front_left_hip_y">
+            <command_interface name="position">
+                <param name="min">-${pi}</param>
+                <param name="max">${pi}</param>
+            </command_interface>
+            <state_interface name="position" />
+            <state_interface name="velocity" />
+            <state_interface name="effort" />
+        </joint>
+        <joint name="front_left_knee">
+            <command_interface name="position">
+                <param name="min">-${pi}</param>
+                <param name="max">${pi}</param>
+            </command_interface>
+            <state_interface name="position" />
+            <state_interface name="velocity" />
+            <state_interface name="effort" />
+        </joint>
+        <joint name="front_right_hip_x">
+            <command_interface name="position">
+                <param name="min">-${pi}</param>
+                <param name="max">${pi}</param>
+            </command_interface>
+            <state_interface name="position" />
+            <state_interface name="velocity" />
+            <state_interface name="effort" />
+        </joint>
+        <joint name="front_right_hip_y">
+            <command_interface name="position">
+                <param name="min">-${pi}</param>
+                <param name="max">${pi}</param>
+            </command_interface>
+            <state_interface name="position" />
+            <state_interface name="velocity" />
+            <state_interface name="effort" />
+        </joint>
+        <joint name="front_right_knee">
+            <command_interface name="position">
+                <param name="min">-${pi}</param>
+                <param name="max">${pi}</param>
+            </command_interface>
+            <state_interface name="position" />
+            <state_interface name="velocity" />
+            <state_interface name="effort" />
+        </joint>
+        <joint name="rear_left_hip_x">
+            <command_interface name="position">
+                <param name="min">-${pi}</param>
+                <param name="max">${pi}</param>
+            </command_interface>
+            <state_interface name="position" />
+            <state_interface name="velocity" />
+            <state_interface name="effort" />
+        </joint>
+        <joint name="rear_left_hip_y">
+            <command_interface name="position">
+                <param name="min">-${pi}</param>
+                <param name="max">${pi}</param>
+            </command_interface>
+            <state_interface name="position" />
+            <state_interface name="velocity" />
+            <state_interface name="effort" />
+        </joint>
+        <joint name="rear_left_knee">
+            <command_interface name="position">
+                <param name="min">-${pi}</param>
+                <param name="max">${pi}</param>
+            </command_interface>
+            <state_interface name="position" />
+            <state_interface name="velocity" />
+            <state_interface name="effort" />
+        </joint>
+        <joint name="rear_right_hip_x">
+            <command_interface name="position">
+                <param name="min">-${pi}</param>
+                <param name="max">${pi}</param>
+            </command_interface>
+            <state_interface name="position" />
+            <state_interface name="velocity" />
+            <state_interface name="effort" />
+        </joint>
+        <joint name="rear_right_hip_y">
+            <command_interface name="position">
+                <param name="min">-${pi}</param>
+                <param name="max">${pi}</param>
+            </command_interface>
+            <state_interface name="position" />
+            <state_interface name="velocity" />
+            <state_interface name="effort" />
+        </joint>
+        <joint name="rear_right_knee">
+             <command_interface name="position">
+                <param name="min">-${pi}</param>
+                <param name="max">${pi}</param>
+            </command_interface>
+            <state_interface name="position" />
+            <state_interface name="velocity" />
+            <state_interface name="effort" />
+        </joint>
+    </ros2_control> -->
+   <gazebo>
+        <plugin name="ign_ros2_control::IgnitionROS2ControlPlugin" filename="ign_ros2_control-system">
             <parameters>$(find champ_bringup)/config/ros2_control_spot.yaml</parameters>
         </plugin>

File: champ_description/urdf/spot/spot_leg.urdf.xacro (robot description, xacro)
@@ -1,10 +1,8 @@
 <?xml version="1.0"?>
 <robot xmlns:xacro="http://ros.org/wiki/xacro">
-    <xacro:arg name="leg_kp" default="400000.0" />
-    <xacro:arg name="leg_kd" default="1.0" />
-    <xacro:arg name="leg_mu" default="0.8" />
-    <xacro:arg name="leg_mu2" default="0.8" />
-    <xacro:arg name="leg_maxVel" default="0.0" />
-    <xacro:arg name="leg_minDepth" default="0.002" />
+    <xacro:arg name="leg_kp" default="1e+07" />
+    <xacro:arg name="leg_kd" default="100.0" />
+    <xacro:arg name="leg_mu1" default="1.0" />
+    <xacro:arg name="leg_mu2" default="1.0" />
     <xacro:arg name="leg_fdir1" default="" />
     <xacro:arg name="max_knee_effort" default="80" />
@@ -14,6 +12,4 @@
     <xacro:arg name="max_hip_y_effort" default="80" />
     <xacro:arg name="max_hip_y_velocity" default="15" />
-    <xacro:arg name="damping" default="0.0" />
-    <xacro:arg name="friction" default="1.0e+07" />
     <xacro:macro name="spot_leg" params="leg_name prefix">
         <xacro:if value="${leg_name == 'front_left'}">
@@ -46,10 +42,8 @@
             <inertial>
                 <mass value="${hip_mass}" />
-                <inertia ixx="${(1/12) * hip_mass * (hip_width * hip_width + hip_height * hip_height)}" ixy="0.0" ixz="0.0"
-                            iyy="${(1/12) * hip_mass * (hip_length * hip_length + hip_height * hip_height)}" iyz="0.0"
-                            izz="${(1/12) * hip_mass * (hip_length * hip_length + hip_width * hip_width)}" />
+                <inertia ixx="${(1/12) * hip_mass * (hip_width * hip_width + hip_height * hip_height)}" ixy="0.0" ixz="0.0" iyy="${(1/12) * hip_mass * (hip_length * hip_length + hip_height * hip_height)}" iyz="0.0" izz="${(1/12) * hip_mass * (hip_length * hip_length + hip_width * hip_width)}" />
             </inertial>
         </link>
-        <joint name="${prefix}${leg_name}_hip_x" type="revolute">
+        <joint name="${leg_name}_hip_x" type="revolute">
             <origin xyz="${base_to_hip_xyz}" rpy="0 0 0" />
             <axis xyz="1 0 0" />
@@ -57,5 +51,5 @@
             <child link="${prefix}${leg_name}_hip" />
             <limit effort="$(arg max_hip_x_effort)" velocity="$(arg max_hip_x_velocity)" lower="-0.78539816339744827899" upper="0.78539816339744827899" />
-            <dynamics damping="$(arg damping)" friction="$(arg friction)" />
+            <dynamics damping="10.0" friction="100.0" />
         </joint>
         <link name="${prefix}${leg_name}_upper_leg">
@@ -66,5 +60,4 @@
             </visual>
             <collision>
-                <origin rpy="0 0 0" xyz="0 0 ${-0.25*upper_leg_height}"/>
                 <geometry>
                     <!-- <mesh filename="file://$(find champ_description)/meshes/spot/${leg_name}_upper_leg_collision.stl" /> -->
@@ -75,10 +68,8 @@
                 <origin xyz="0 0 -0.14" rpy="0 0 0" />
                 <mass value="${upper_leg_mass}" />
-                <inertia ixx="${(1/12) * upper_leg_mass * (upper_leg_width * upper_leg_width + upper_leg_height * upper_leg_height)}" ixy="0.0" ixz="0.0"
-                            iyy="${(1/12) * upper_leg_mass * (upper_leg_length * upper_leg_length + upper_leg_height * upper_leg_height)}" iyz="0.0"
-                            izz="${(1/12) * upper_leg_mass * (upper_leg_length * upper_leg_length + upper_leg_width * upper_leg_width)}" />
+                <inertia ixx="${(1/12) * upper_leg_mass * (upper_leg_width * upper_leg_width + upper_leg_height * upper_leg_height)}" ixy="0.0" ixz="0.0" iyy="${(1/12) * upper_leg_mass * (upper_leg_length * upper_leg_length + upper_leg_height * upper_leg_height)}" iyz="0.0" izz="${(1/12) * upper_leg_mass * (upper_leg_length * upper_leg_length + upper_leg_width * upper_leg_width)}" />
             </inertial>
         </link>
-        <joint name="${prefix}${leg_name}_hip_y" type="revolute">
+        <joint name="${leg_name}_hip_y" type="revolute">
             <origin xyz="${hip_to_upper_leg_xyz}" rpy="0 0 0" />
             <axis xyz="0 1 0" />
@@ -86,5 +77,5 @@
             <child link="${prefix}${leg_name}_upper_leg" />
             <limit effort="$(arg max_hip_y_effort)" velocity="$(arg max_hip_y_velocity)" lower="-0.89884456477707963539" upper="2.2951079663725435509" />
-            <dynamics damping="$(arg damping)" friction="$(arg friction)" />
+            <dynamics damping="10.0" friction="100.0" />
         </joint>
         <link name="${prefix}${leg_name}_lower_leg">
@@ -95,8 +86,13 @@
             </visual>
             <collision>
-                <origin rpy="0 0 0" xyz="0 0 ${-0.35*lower_leg_height}"/>
                 <geometry>
                     <!-- <mesh filename="file://$(find champ_description)/meshes/spot/${leg_name}_lower_leg_collision.stl" scale="0.82 0.97 0.98" /> -->
                     <cylinder radius="${lower_leg_length}" length="${0.6*lower_leg_height}"/>
+                </geometry>
+            </collision>
+            <collision>
+                <origin xyz="0 0 -${lower_leg_to_foot_z - 0.04 + 0.003}" />
+                <geometry>
+                    <sphere radius="0.04" />
                 </geometry>
             </collision>
@@ -104,40 +100,12 @@
                 <origin xyz="0 0 -0.16" rpy="0 0 0" />
                 <mass value="${lower_leg_mass}" />
-                <inertia ixx="${(1/12) * lower_leg_mass * (lower_leg_width * lower_leg_width + lower_leg_height * lower_leg_height)}" ixy="0.0" ixz="0.0"
-                         iyy="${(1/12) * lower_leg_mass * (lower_leg_length * lower_leg_length + lower_leg_height * lower_leg_height)}" iyz="0.0"
-                         izz="${(1/12) * lower_leg_mass * (lower_leg_length * lower_leg_length + lower_leg_width * lower_leg_width)}" />
+                <inertia ixx="${(1/12) * lower_leg_mass * (lower_leg_width * lower_leg_width + lower_leg_height * lower_leg_height)}" ixy="0.0" ixz="0.0" iyy="${(1/12) * lower_leg_mass * (lower_leg_length * lower_leg_length + lower_leg_height * lower_leg_height)}" iyz="0.0" izz="${(1/12) * lower_leg_mass * (lower_leg_length * lower_leg_length + lower_leg_width * lower_leg_width)}" />
             </inertial>
         </link>
-        <joint name="${prefix}${leg_name}_knee" type="revolute">
-            <origin xyz="${upper_leg_to_lower_leg_x} 0 -${upper_leg_to_lower_leg_z}" rpy="0 0 0" />
-            <axis xyz="0 1 0" />
-            <parent link="${prefix}${leg_name}_upper_leg" />
-            <child link="${prefix}${leg_name}_lower_leg" />
-            <limit effort="$(arg max_knee_effort)" velocity="$(arg max_knee_velocity)" lower="-2.7929" upper="-0.254801" />
-            <dynamics damping="$(arg damping)" friction="$(arg friction)" />
-        </joint>
-        <!-- <xacro:empty_link name="${prefix}${leg_name}_ee" /> -->
-        <link name="${prefix}${leg_name}_ee">
-            <collision name="${prefix}${leg_name}_ee_collision">
-                <origin rpy="0 0 0" xyz="0 0 ${lower_leg_length}"/>
-                <geometry>
-                    <sphere radius="${lower_leg_length}"/>
-                </geometry>
-            </collision>
-        </link>
-        <joint name="${prefix}${leg_name}_foot" type="fixed">
-            <parent link="${prefix}${leg_name}_lower_leg" />
-            <child link="${prefix}${leg_name}_ee" />
-            <origin xyz="0 0 -${lower_leg_to_foot_z}" rpy="0 0 0" />
-            <limit effort="$(arg max_knee_effort)" velocity="$(arg max_knee_velocity)" lower="-2.7929" upper="-0.254801" />
-            <dynamics damping="$(arg damping)" friction="$(arg friction)" />
-        </joint>
-        <gazebo reference="${prefix}${leg_name}_ee">
+        <gazebo reference="${prefix}${leg_name}_lower_leg">
             <kp>$(arg leg_kp)</kp>
             <kd>$(arg leg_kd)</kd>
-            <mu>$(arg leg_mu)</mu>
+            <mu1>$(arg leg_mu1)</mu1>
             <mu2>$(arg leg_mu2)</mu2>
-            <maxVel>$(arg leg_maxVel)</maxVel>
-            <minDepth>$(arg leg_minDepth)</minDepth>
             <xacro:if value="${'$(arg leg_fdir1)' != ''}">
                 <fdir1>$(arg leg_fdir1)</fdir1>
@@ -149,34 +117,17 @@
                 </contact>
             </sensor>
-            <maxContacts>1</maxContacts>
-            <minDepth>0.005</minDepth>
-            <gravity>true</gravity>
-            <collision name="${prefix}${leg_name}_ee_collision">
-                <geometry>
-                    <sphere>
-                        <!-- should be the same as surface_radius -->
-                        <radius>0.02175</radius>
-                    </sphere>
-                </geometry>
-            <surface>
-                <friction>
-                    <torsional>
-                        <coefficient>10</coefficient>
-                        <use_patch_radius>true</use_patch_radius>
-                        <!-- should be the same as collision sphere radius -->
-                        <surface_radius>0.02175</surface_radius>
-                        <patch_radius>0.01</patch_radius>
-                    </torsional>
-                </friction>
-                <contact>
-                    <poissons_ratio>0.5</poissons_ratio>
-                    <elastic_modulus>1e8</elastic_modulus>
-                </contact>
-            </surface>
-            </collision>
-            <material>Gazebo/Black</material>
         </gazebo>
+        <joint name="${leg_name}_knee" type="revolute">
+            <origin xyz="${upper_leg_to_lower_leg_x} 0 -${upper_leg_to_lower_leg_z}" rpy="0 0 0" />
+            <axis xyz="0 1 0" />
+            <parent link="${prefix}${leg_name}_upper_leg" />
+            <child link="${prefix}${leg_name}_lower_leg" />
+            <limit effort="$(arg max_knee_effort)" velocity="$(arg max_knee_velocity)" lower="-2.7929" upper="-0.254801" />
+            <dynamics damping="10.0" friction="100.0" />
+        </joint>
+        <xacro:empty_link name="${prefix}${leg_name}_ee" />
+        <xacro:fixed_joint name="${leg_name}_foot" parent="${prefix}${leg_name}_lower_leg" child="${prefix}${leg_name}_ee" xyz="0 0 -${lower_leg_to_foot_z}" />
         <!-- Not actually used now, but doesn't hurt to have it here ready for future use with ros_ign_control. -->
-        <transmission name="${leg_name}_hip_x_trans">
+        <!-- <transmission name="${leg_name}_hip_x_trans">
             <type>transmission_interface/SimpleTransmission</type>
             <joint name="${leg_name}_hip_x">
@@ -207,8 +158,8 @@
                 <mechanicalReduction>1</mechanicalReduction>
             </actuator>
-        </transmission>
-        <ros2_control name="${leg_name}_GazeboSystem" type="system">
+        </transmission> -->
+        <ros2_control name="${leg_name}_IgnitionSystem" type="system">
             <hardware>
-                <plugin>gazebo_ros2_control/GazeboSystem</plugin>
+                <plugin>ign_ros2_control/IgnitionSystem</plugin>
             </hardware>
             <joint name="${leg_name}_hip_x">
